File: PCBProject_InverterFNC42060F/Kicad_inverter/inverter/inverter.kicad_sch (KiCad schematic)
At the start: 104 parts, among them IC1 TLP2270_D4-LF4,E, IC2 TLP2270_D4-LF4,E, IC3 TLP2270_D4-LF4,E, J1 Conn_02x06_Top_Bottom, J10 Conn_01x06_Pin, J11 Header 2, J12 Conn_02x02_Odd_Even, J2 board_1, J3 board_1, J4 Conn_01x02_Pin, J5 Conn_01x02_Pin, J6 Header 2, J7 Header 2, J8 Header 2, J9 Header 2, Q1 FMMT618TA, Q2 FNC42060F, U1 VIPER22A, U2 LM2675M-5.0

Commit message: update inverter board
Parts:
- added J13: Conn_01x02_Pin, Connector_PinSocket_2.54mm:PinSocket_1x02_P2.54mm_Vertical, symbol Connector:Conn_01x02_Pin
Connections:
- net GND: now also J13.2 (Pin_2)
- net TEMP1: now also J13.1 (Pin_1)
Other:
- moved on the sheet: C34, C35, C36, C37, C38, C39, D6, L2, U2
