File: PCBProject_InverterFNC42060F/Kicad_inverter/inverter/inverter_board1.kicad_pcb (KiCad board)
At the start: 4 copper layers, 100 x 50 mm, 56 parts, among them IC1 TLP2270_D4-LF4,E, IC2 TLP2270_D4-LF4,E, IC3 TLP2270_D4-LF4,E, J1 Conn_02x06_Top_Bottom, J12 Conn_02x02_Odd_Even, J2 board_1, J4 Conn_01x02_Pin, J5 Conn_01x02_Pin, J6 Header 2, J7 Header 2, U1 VIPER22A, U2 LM2675M-5.0

Commit message: update inverter board
Routing:
- net GND: vias 34 -> 53
Changed lines of the file:
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@@
     )
   )
-  (gr_rect (start 78.400002 91.575) (end 93.150002 86.325)
+  (gr_rect (start 78.400002 86.325) (end 93.150002 91.575)
     (stroke (width 0.1) (type default)) (fill none) (layer "B.SilkS"))
   (gr_arc (start 127 89) (mid 123 85) (end 127 81)
@@
   (segment (start 68 84.5) (end 70.45 84.5) (width 0.5) (layer "F.Cu") (net 1))
   (segment (start 74.45 85.825) (end 76.175 85.825) (width 0.5) (layer "F.Cu") (net 1))
+  (segment (start 63.7 82.4) (end 65.9 82.4) (width 0.5) (layer "F.Cu") (net 1))
   (segment (start 59.375 110.583) (end 61.083 110.583) (width 0.3) (layer "F.Cu") (net 1))
   (segment (start 61.083 110.583) (end 61.1 110.6) (width 0.3) (layer "F.Cu") (net 1))
@@
   (segment (start 47.145 73.655) (end 47.145 74.895) (width 0.5) (layer "F.Cu") (net 1))
   (segment (start 92.119501 92.880499) (end 103 92.880499) (width 5) (layer "F.Cu") (net 1))
-  (segment (start 62.25 82.4) (end 65.9 82.4) (width 0.5) (layer "F.Cu") (net 1))
+  (segment (start 62.25 82.4) (end 63.7 82.4) (width 0.5) (layer "F.Cu") (net 1))
   (segment (start 74.325 85.7) (end 74.45 85.825) (width 0.5) (layer "F.Cu") (net 1))
   (segment (start 60.981 94.581) (end 61 94.6) (width 0.3) (layer "F.Cu") (net 1))
@@
   (via (at 75 68) (size 0.5) (drill 0.3) (layers "F.Cu" "B.Cu") (free) (net 1))
   (via (at 64 67) (size 0.5) (drill 0.3) (layers "F.Cu" "B.Cu") (free) (net 1))
+  (via (at 59.3 74.4) (size 0.6) (drill 0.3) (layers "F.Cu" "B.Cu") (free) (net 1))
+  (via (at 60.8 82.4) (size 0.6) (drill 0.3) (layers "F.Cu" "B.Cu") (free) (net 1))
   (via (at 76.2 85.8) (size 0.7) (drill 0.5) (layers "F.Cu" "B.Cu") (net 1))
+  (via (at 59.2 76.7) (size 0.6) (drill 0.3) (layers "F.Cu" "B.Cu") (free) (net 1))
   (via (at 63 67) (size 0.5) (drill 0.3) (layers "F.Cu" "B.Cu") (free) (net 1))
   (via (at 75 69) (size 0.5) (drill 0.3) (layers "F.Cu" "B.Cu") (free) (net 1))
@@
   (via (at 71.6 87.1) (size 0.7) (drill 0.5) (layers "F.Cu" "B.Cu") (net 1))
   (via (at 65 67) (size 0.5) (drill 0.3) (layers "F.Cu" "B.Cu") (free) (net 1))
+  (via (at 73.2 68.2) (size 0.6) (drill 0.3) (layers "F.Cu" "B.Cu") (free) (net 1))
   (via (at 68 67) (size 0.5) (drill 0.3) (layers "F.Cu" "B.Cu") (free) (net 1))
   (via (at 61.1 110.6) (size 0.5) (drill 0.3) (layers "F.Cu" "B.Cu") (net 1))
@@
   (via (at 74 67) (size 0.5) (drill 0.3) (layers "F.Cu" "B.Cu") (free) (net 1))
   (via (at 61 79.2) (size 0.5) (drill 0.3) (layers "F.Cu" "B.Cu") (free) (net 1))
+  (via (at 68.2 68.3) (size 0.6) (drill 0.3) (layers "F.Cu" "B.Cu") (free) (net 1))
+  (via (at 55.1 75.2) (size 0.6) (drill 0.3) (layers "F.Cu" "B.Cu") (free) (net 1))
   (via (at 62 67) (size 0.5) (drill 0.3) (layers "F.Cu" "B.Cu") (free) (net 1))
+  (via (at 65.6 68.3) (size 0.6) (drill 0.3) (layers "F.Cu" "B.Cu") (free) (net 1))
+  (via (at 77.3 73.4) (size 0.6) (drill 0.3) (layers "F.Cu" "B.Cu") (free) (net 1))
   (via (at 75 67) (size 0.5) (drill 0.3) (layers "F.Cu" "B.Cu") (free) (net 1))
+  (via (at 52.3 75.2) (size 0.6) (drill 0.3) (layers "F.Cu" "B.Cu") (free) (net 1))
   (via (at 60 67) (size 0.5) (drill 0.3) (layers "F.Cu" "B.Cu") (free) (net 1))
   (via (at 61.1 102.4) (size 0.5) (drill 0.3) (layers "F.Cu" "B.Cu") (net 1))
   (via (at 63.4 89.2) (size 0.5) (drill 0.3) (layers "F.Cu" "B.Cu") (net 1))
+  (via (at 77.7 71.1) (size 0.6) (drill 0.3) (layers "F.Cu" "B.Cu") (free) (net 1))
   (via (at 61 94.6) (size 0.5) (drill 0.3) (layers "F.Cu" "B.Cu") (net 1))
+  (via (at 70.6 68.3) (size 0.6) (drill 0.3) (layers "F.Cu" "B.Cu") (free) (net 1))
   (via (at 62.2 104) (size 0.5) (drill 0.3) (layers "F.Cu" "B.Cu") (net 1))
   (via (at 71 67) (size 0.5) (drill 0.3) (layers "F.Cu" "B.Cu") (free) (net 1))
   (via (at 73 67) (size 0.5) (drill 0.3) (layers "F.Cu" "B.Cu") (free) (net 1))
+  (via (at 62.9 68.3) (size 0.6) (drill 0.3) (layers "F.Cu" "B.Cu") (free) (net 1))
   (via (at 72 67) (size 0.5) (drill 0.3) (layers "F.Cu" "B.Cu") (free) (net 1))
   (via (at 68 86.5) (size 0.7) (drill 0.5) (layers "F.Cu" "B.Cu") (net 1))
+  (via (at 81.4 74.6) (size 0.6) (drill 0.3) (layers "F.Cu" "B.Cu") (free) (net 1))
   (via (at 56.3 79.35) (size 0.5) (drill 0.3) (layers "F.Cu" "B.Cu") (free) (net 1))
+  (via (at 57.8 82.3) (size 0.6) (drill 0.3) (layers "F.Cu" "B.Cu") (free) (net 1))
+  (via (at 57.8 78.1) (size 0.6) (drill 0.3) (layers "F.Cu" "B.Cu") (free) (net 1))
+  (via (at 77.7 67.7) (size 0.6) (drill 0.3) (layers "F.Cu" "B.Cu") (free) (net 1))
+  (via (at 60.3 68.3) (size 0.6) (drill 0.3) (layers "F.Cu" "B.Cu") (free) (net 1))
+  (via (at 77.3 74.6) (size 0.6) (drill 0.3) (layers "F.Cu" "B.Cu") (free) (net 1))
   (via (at 69 67) (size 0.5) (drill 0.3) (layers "F.Cu" "B.Cu") (free) (net 1))
   (via (at 70 67) (size 0.5) (drill 0.3) (layers "F.Cu" "B.Cu") (free) (net 1))
@@
   (via (at 56.15 76.85) (size 0.5) (drill 0.3) (layers "F.Cu" "B.Cu") (free) (net 1))
   (via (at 57.25 75.5) (size 0.5) (drill 0.3) (layers "F.Cu" "B.Cu") (free) (net 1))
+  (via (at 63.7 82.4) (size 0.6) (drill 0.3) (layers "F.Cu" "B.Cu") (net 1))
   (via (at 61 67) (size 0.5) (drill 0.3) (layers "F.Cu" "B.Cu") (free) (net 1))
   (via (at 47.95 69.9) (size 0.5) (drill 0.3) (layers "F.Cu" "B.Cu") (net 1))
@@
   (segment (start 127 97) (end 120.5 97) (width 5) (layer "F.Cu") (net 3))
   (segment (start 95.819501 102.880499) (end 91.7 107) (width 5) (layer "F.Cu") (net 3))
+  (segment (start 59.285 92.041) (end 65.041 92.041) (width 0.3) (layer "F.Cu") (net 4))
+  (segment (start 72.1 113.9) (end 72 114) (width 0.3) (layer "F.Cu") (net 4))
+  (segment (start 72.1 99.1) (end 72.1 113.9) (width 0.3) (layer "F.Cu") (net 4))
   (segment (start 65.041 92.041) (end 72.1 99.1) (width 0.3) (layer "F.Cu") (net 4))
-  (segment (start 72 111.7) (end 72 114) (width 0.3) (layer "F.Cu") (net 4))
-  (segment (start 72.1 111.6) (end 72 111.7) (width 0.3) (layer "F.Cu") (net 4))
-  (segment (start 59.285 92.041) (end 65.041 92.041) (width 0.3) (layer "F.Cu") (net 4))
-  (segment (start 72.1 99.1) (end 72.1 111.6) (width 0.3) (layer "F.Cu") (net 4))
   (segment (start 59.285 93.311) (end 62.711 93.311) (width 0.3) (layer "F.Cu") (net 5))
   (segment (start 62.711 93.311) (end 69.5 100.1) (width 0.3) (layer "F.Cu") (net 5))
@@
         (xy 96.561638 106.188362)
         (xy 93.8 108.95)
-        (xy 93.8 108.95)
         (xy 92.45 110.5)
