File: PCBProject_InverterFNC42060F/Kicad_inverter/inverter/inverter_board2.kicad_pcb (KiCad board)
At the start: 4 copper layers, 53 x 50 mm, 47 parts, among them J10 Conn_01x06_Pin, J11 Header 2, J12 Conn_02x02_Odd_Even, J3 board_1, J8 Header 2, J9 Header 2, Q1 FMMT618TA, Q2 FNC42060F

Commit message: update inverter board
Parts:
- added J13: Conn_01x02_Pin, Connector_PinSocket_2.54mm:PinSocket_1x02_P2.54mm_Vertical, F.Cu at (56.3, 113.1)
Routing:
- net /TEMP1: track 5.14 -> 27.9 mm, vias 0 -> 2
- net /W: track 34.0 -> 35.2 mm
- net Net-(Q2-CSC): track 24.9 -> 24.1 mm
- net /V: track 30.1 -> 29.6 mm
- net /OPWM3B: track 14.4 -> 13.9 mm
- net GND: vias 14 -> 30
- added copper zone on B.Cu, net /V
