File: PCBProject_Extension28377dBGA/Extension/sheet1.kicad_sch (KiCad schematic)
At the start: 259 parts, among them J1 HIF3FC-20PA-2.54DSA, J12 HIF3FC-20PA-2.54DSA, J17 HIF3FC-20PA-2.54DSA, J2 HIF3FC-20PA-2.54DSA, J3 HIF3FC-20PA-2.54DSA, J4 HIF3FC-10PA-2.54DSA, J5 HIF3FC-10PA-2.54DSA, J9 HIF3FC-20PA-2.54DSA, P1 TMS320F28377D-BGA-Core, P10 Header 2X2, P11 Header 2X2, P12 Header 2X2, P2 Header 6X2, P3 Header 2X2, P4 Header 2X2, P5 Header 2X2, P6 Header 2X2, P7 Header 2X2, P8 Header 2X2, P9 Header 2X2, Q1 FMMT618TA, Q2 FMMT618TA, Q3 FMMT618TA, Q4 FMMT618TA, U1 SN74HC365D, U6 ${MANUFACTURER PART}, U7 ${MANUFACTURER PART}

Commit message: update sheet1 (kicad)
Parts:
- removed J5: HIF3FC-10PA-2.54DSA, D:_horyc_Documents_AltiumLL_SamacSys.PcbLib_SHDR10W50P254_2X5_2020X850X920P, symbol sheet1-altium-import:root_0_HIF3FC-10PA-2.54DSA
- removed J9: HIF3FC-20PA-2.54DSA, D:_horyc_Documents_AltiumLL_SamacSys.PcbLib_SHDR20W56P254_2X10_3290X850X950P, symbol sheet1-altium-import:root_0_HIF3FC-20PA-2.54DSA
- removed P3, P4, P5, P6, P7, P8: Header 2X2, HDR2X2, symbol sheet1-altium-import:root_0_Header 2X2
- removed TP8: AGND 黑色测试点, TP, symbol sheet1-altium-import:root_0_测试点
- added CAN1, CAN2, SPI2, UART1, UART2, UART3, UART4: Conn_02x04_Counter_Clockwise, symbol Connector_Generic:Conn_02x04_Counter_Clockwise
- gave numbers to parts that had none: 164
- renumbered J12 to SPI1
Connections:
- net VCO_ECAP4 is gone; now on net ECAP4_IPM_TerminalDutyU2: P1.90 (A16_90)
- net VCO_ECAP5 is gone; now on net ECAP5_IPM_TerminalDutyV2: P1.92 (A15_92)
- net VCO_ECAP6 is gone; now on net ECAP6_IPM_TerminalDutyW2: P1.94 (A14_94)
- net AGND: now also J17.2, J17.4, CAN1.5 (Pin_5), CAN1.6 (Pin_6), CAN2.5 (Pin_5), CAN2.6 (Pin_6), SPI2.5 (Pin_5), SPI2.6 (Pin_6), UART1.5 (Pin_5), UART1.6 (Pin_6), UART2.5 (Pin_5), UART2.6 (Pin_6), UART3.5 (Pin_5), UART3.6 (Pin_6), UART4.5 (Pin_5), UART4.6 (Pin_6); no longer POWER1.19, POWER1.20
- net D+5V: now also J17.11, J17.9, CAN1.3 (Pin_3), CAN1.4 (Pin_4), CAN2.3 (Pin_3), CAN2.4 (Pin_4), SPI2.3 (Pin_3), SPI2.4 (Pin_4), UART1.3 (Pin_3), UART1.4 (Pin_4), UART2.3 (Pin_3), UART2.4 (Pin_4), UART3.3 (Pin_3), UART3.4 (Pin_4), UART4.3 (Pin_3), UART4.4 (Pin_4)
- net DC_BUS_2M1: no longer P22.1, P22.2, P22.3, P22.4, R76.2
- net DSP_A_CAN_RX: now also CAN2.8 (Pin_8)
- net DSP_A_CAN_TX: now also CAN2.7 (Pin_7)
- net DSP_B_CAN_RX: now also CAN1.8 (Pin_8)
- net DSP_B_CAN_TX: now also CAN1.7 (Pin_7)
- net GND_2M1: no longer P21.1, P21.2, P21.3, P21.4, R75.2
- net IPM_VDC_BUS1: now also C39.2, D24.3, R88.2, TP32.1
- net IPM_VDC_BUS2: no longer C39.2, D24.3, R88.2, TP32.1
- net SPI B MI HS: now also SPI2.2 (Pin_2)
- net SPI B MO HS: now also SPI2.1 (Pin_1)
- net SPI_B_CK_HS: now also SPI2.8 (Pin_8)
- net UART_SCI_RXDA: now also UART1.8 (Pin_8)
- net UART_SCI_RXDB: now also UART2.7 (Pin_7)
- net UART_SCI_RXDC: now also UART3.8 (Pin_8)
- net UART_SCI_RXDD: now also UART4.7 (Pin_7)
- net UART_SCI_TXDA: now also UART1.7 (Pin_7)
- net UART_SCI_TXDB: now also UART2.8 (Pin_8)
- net UART_SCI_TXDC: now also UART3.7 (Pin_7)
- net UART_SCI_TXDD: now also UART4.8 (Pin_8)
- net VDD: now also CAN1.1 (Pin_1), CAN1.2 (Pin_2), CAN2.1 (Pin_1), CAN2.2 (Pin_2)
- net ~{SPI_B_STE_HS}: now reaches P1.148 (GP143_148)
- net ~{SPI_B_STE_HS}: now also SPI2.7 (Pin_7)
- net IPM_TerminalDutyU1 renamed ECAP1_IPM_TerminalDutyU1
- net ECAP1_IPM_TerminalDutyU1: now also P1.84 (A19_84)
- net IPM_TerminalDutyV1 renamed ECAP2_IPM_TerminalDutyV1
- net ECAP2_IPM_TerminalDutyV1: now also P1.86 (A18_86)
- net IPM_TerminalDutyW1 renamed ECAP3_IPM_TerminalDutyW1
- net ECAP3_IPM_TerminalDutyW1: now also P1.88 (A17_88)
- net VCO_ECAP1 renamed ECAP6_IPM_TerminalDutyW2
- net ECAP6_IPM_TerminalDutyW2: no longer P1.84 (A19_84)
- net VCO_ECAP2 renamed ECAP5_IPM_TerminalDutyV2
- net ECAP5_IPM_TerminalDutyV2: no longer P1.86 (A18_86)
- net VCO_ECAP3 renamed ECAP4_IPM_TerminalDutyU2
- net ECAP4_IPM_TerminalDutyU2: no longer P1.88 (A17_88)
- net \~{SPI_C_STE_H}S renamed ~{SPI_C_STE_HS}
- new net D12V1: POWER1.19, POWER1.20, UART1.1 (Pin_1), UART1.2 (Pin_2), UART2.1 (Pin_1), UART2.2 (Pin_2), UART3.1 (Pin_1), UART3.2 (Pin_2), UART4.1 (Pin_1), UART4.2 (Pin_2)
- new net DC_BUS_2M2: P22.1, P22.2, P22.3, P22.4, R76.2
- new net GND_2M2: P21.1, P21.2, P21.3, P21.4, R75.2
- no-connect marks 99 -> 96
Other:
- moved on the sheet: C1, C2, C3, C4, C5, C6, C7, J1, J2, J3, J4, P2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

Commit message: Add sheet pcb.
Parts:
- C1, C10, C11, C12, C13, C14, C15, C16, C17, C18, C19, C2, C20, C21, C22, C23, C24, C25, C26, C27, C28, C29, C3, C30, C31, C32, C33, C34, C35, C36, C37, C38, C39, C4, C40, C41, C5, C6, C7, C8, C9, R1, R10, R11, R12, R13, R14, R2, R3, R30, R31, R32, R33, R34, R35, R37, R38, R39, R4, R40, R45, R46, R49, R5, R50, R51, R52, R53, R54, R55, R56, R59, R6, R60, R61, R62, R63, R64, R65, R66, R67, R68, R69, R7, R70, R71, R72, R73, R74, R75, R76, R77, R78, R79, R8, R80, R81, R82, R83, R84, R85, R86, R87, R88, R89, R9, R90, R91, R92, R93, R94, RU1, RU2, RU3, RU4, RU5: footprint 0805 -> mmlab-footprint-library:0805
- CAN1, CAN2, SPI2, UART1, UART2, UART3, UART4: footprint (none) -> Connector_PinSocket_2.54mm:PinSocket_2x04_P2.54mm_Vertical
- D1, D2, D30, D31: footprint L0805 -> mmlab-footprint-library:L0805
- D10, D11, D12, D13, D14, D15, D16, D17, D18, D19, D20, D21, D22, D23, D24, D25, D26, D3, D4, D5, D6, D7, D8, D9, Q1, Q2, Q3, Q4: footprint SOT-23 -> Package_TO_SOT_SMD:SOT-23
- J1, J17, J2, J3, SPI1: footprint D:_horyc_Documents_AltiumLL_SamacSys.PcbLib_SHDR20W56P254_2X10_3290X850X950P -> Connector_IDC:IDC-Header_2x10_P2.54mm_Vertical
- J4, TMP1: footprint D:_horyc_Documents_AltiumLL_SamacSys.PcbLib_SHDR10W50P254_2X5_2020X850X920P -> Connector_IDC:IDC-Header_2x05_P2.54mm_Vertical
- LEM1, LEM2, LEM3, LEM4: footprint D:_codefile_ProjectEureka_ProjectEureka_Project_Oshinoko.PcbLib_SHDR30W50P254_2X15_4560X850X1200P -> Connector_IDC:IDC-Header_2x15_P2.54mm_Vertical
- N1, N2: footprint SOIC14_M -> mmlab-footprint-library:SOIC14_M
- P1: footprint DSP_240_0p6mm -> mmlab-footprint-library:DSP_240
- P10, P11, P12, P17, P18, P19, P20, P21, P22, P23, P24, P9: footprint HDR2X2 -> Connector_PinSocket_2.54mm:PinSocket_2x02_P2.54mm_Vertical
- P13, P14, P15, P16, P2: footprint HDR2X6 -> Connector_PinSocket_2.54mm:PinSocket_2x06_P2.54mm_Vertical
- POWER1: footprint HDR2.54-LI-2x15P -> Connector_PinSocket_2.54mm:PinSocket_2x15_P2.54mm_Vertical
- R15, R16, R17, R18, R19, R20, R21, R22, R23, R24, R25, R26, R27, R28, R29, R36, R41, R42, R43, R44, R47, R48, R57, R58: footprint 0805 -> Resistor_SMD:R_0402_1005Metric
- TP1, TP10, TP11, TP12, TP13, TP14, TP15, TP16, TP17, TP18, TP19, TP2, TP20, TP21, TP22, TP23, TP24, TP25, TP26, TP27, TP28, TP29, TP3, TP30, TP31, TP32, TP33, TP34, TP4, TP5, TP6, TP7, TP9, U6, U7: footprint TESTPOINT-TH_BD1.0 -> mmlab-footprint-library:TESTPOINT-TH_BD1.0
- U1: footprint D016_N -> mmlab-footprint-library:D016_N
- U2, U3, U4, U5: footprint TSSOP-20 -> mmlab-footprint-library:TSSOP-20
Connections:
- net at C14.2, D5.3, R12.2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: now also N1.10; no longer N2.10
- net at C18.2, R65.1, R69.2: now also N1.8; no longer N2.8
- net at C18.1, R39.1, R65.2: now also N1.9; no longer N2.9
- net at C36.2, R86.2, R90.1: now also N2.8; no longer N1.8
- net at C36.1, R77.1, R86.1: now also N2.9; no longer N1.9
- net at C32.2, R78.1, R82.2: now also N2.10; no longer N1.10
