File: PCBProject_Extension28377dBGA/Extension/sheet1.kicad_pcb (KiCad board)
At the start: 4 copper layers, 251 parts, among them J1 HIF3FC-20PA-2.54DSA, J17 HIF3FC-20PA-2.54DSA, J2 HIF3FC-20PA-2.54DSA, J3 HIF3FC-20PA-2.54DSA, J4 HIF3FC-10PA-2.54DSA, P1 TMS320F28377D-BGA-Core, P10 Header 2X2, P11 Header 2X2, P12 Header 2X2, P13 Header 6X2, P14 Header 6X2, P15 Header 6X2, P16 Header 6X2, P17 Header 2X2, P18 Header 2X2, P19 Header 2X2, P2 Header 6X2, P20 Header 2X2, P21 Header 2X2, P22 Header 2X2, P23 Header 2X2, P24 Header 2X2, P9 Header 2X2, Q1 FMMT618TA, Q2 FMMT618TA, Q3 FMMT618TA, Q4 FMMT618TA, U1 SN74HC365D, U2 SN74ABT541, U3 SN74ABT541, U4 SN74ABT541, U5 SN74ABT541, U6 TP-黄色测试点, U7 TP-黄色测试点

Commit message: Place the components.
Parts:
- C25, C26, C8, C9, U2, U3, U4: moved to F.Cu
- P10, P11, P12, P9, POWER1: moved to B.Cu
- moved C13 534.9 mm to (321.4, 182.1), turned to 90 degrees
- moved R11 532.4 mm to (332.3, 183.2), turned to 90 degrees
- moved D4 519.6 mm to (342.5, 188.1), turned to 90 degrees
- moved C22 515.6 mm to (306.2, 177.5), turned to 90 degrees
- moved R68 513.0 mm to (331.4, 187.5), turned to 90 degrees
- moved R64 501.8 mm to (319.2, 187.5), turned to 90 degrees
- moved C17 501.7 mm to (290.9, 177.5), turned to 90 degrees
- moved SPI1 495.2 mm to (270.3, 223.3)
- moved R60 491.0 mm to (307.0, 187.5), turned to 90 degrees
- moved R38 491.0 mm to (300.7, 171.5), turned to 90 degrees
- moved RU4 490.8 mm to (271.5, 212.9)
- moved N1 489.5 mm to (329.0, 171.4), turned to 90 degrees
- moved D1 468.2 mm to (210.6, 154.4)
- moved D2 468.2 mm to (210.6, 157.8)
- moved D31 468.2 mm to (210.6, 164.7)
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