File: PCBProject_Extension28377dBGA/ExtensionSimple/sheet1.kicad_sch (KiCad schematic)
At the start: 118 parts, among them J1 HIF3FC-20PA-2.54DSA, J17 HIF3FC-20PA-2.54DSA, J2 HIF3FC-20PA-2.54DSA, J3 HIF3FC-20PA-2.54DSA, P1 TMS320F28377D-BGA-Core, P10 Header 2X2, P11 Header 2X2, P12 Header 2X2, P13 Header 6X2, P14 Header 6X2, P19 Header 2X2, P2 Header 6X2, P20 Header 2X2, P21 Header 2X2, P22 Header 2X2, P9 Header 2X2, Q2 FMMT618TA, U1 SN74HC365D, U2 SN74ABT541, U3 SN74ABT541

Commit message: fix bugs in power and LEM boards
12VGND should be negative input to amp on LEM. May be also need single connected?
Parts:
- removed C1, C3, C5: 101, mmlab-footprint-library:0805, symbol sheet1-altium-import:root_3_Cap
- removed C6: 103, mmlab-footprint-library:0805, symbol sheet1-altium-import:root_3_Cap
- removed J3: HIF3FC-20PA-2.54DSA, Connector_IDC:IDC-Header_2x10_P2.54mm_Vertical, symbol sheet1-altium-import:root_0_HIF3FC-20PA-2.54DSA
- removed P2: Header 6X2, Connector_PinSocket_2.54mm:PinSocket_2x06_P2.54mm_Vertical, symbol sheet1-altium-import:root_0_Header 6X2
- removed R3, R4, R5, R7: 1K, mmlab-footprint-library:0805, symbol sheet1-altium-import:root_1_Res2
- removed U1: SN74HC365D, mmlab-footprint-library:D016_N, symbol sheet1-altium-import:root_0_SN74HC365D
- added DI1: Conn_02x02_Counter_Clockwise, Connector_PinSocket_2.54mm:PinSocket_2x02_P2.54mm_Vertical, symbol Connector_Generic:Conn_02x02_Counter_Clockwise
- added U4: SN74HC365D, 1mmlab_footprint:SOIC127P600X175-16N, symbol 1mmlab:SN74HC365D
- AGND1: renamed from TP7; footprint mmlab-footprint-library:TESTPOINT-TH_BD1.0 -> TestPoint:TestPoint_Pad_2.0x2.0mm
- C2, C25, C26, C30, C31, C34, C35, C37, C39, C4, C40, C7, C8, C9: footprint mmlab-footprint-library:0805 -> Capacitor_SMD:C_0402_1005Metric
- D1: footprint mmlab-footprint-library:L0805 -> LED_SMD:LED_0805_2012Metric
- N2: footprint mmlab-footprint-library:SOIC14_M -> 1mmlab_footprint:SOIC14_M
- P1: footprint mmlab-footprint-library:DSP_240 -> 1mmlab_footprint:DSP_240
- R1, R2, R30, R32, R34, R8, R80, R81, R84, R85, R88, R89, R9, R91, R92, R93, R94: footprint mmlab-footprint-library:0805 -> Resistor_SMD:R_0402_1005Metric
- R13: value 3,.3K -> 3.3K/1%; footprint mmlab-footprint-library:0805 -> Resistor_SMD:R_0402_1005Metric
- R55, R56, R73, R74, R75, R76, RU1, RU4, RU5: footprint mmlab-footprint-library:0805 -> Resistor_SMD:R_0805_2012Metric
- R6: value 1.69K -> 1.69K/1%; footprint mmlab-footprint-library:0805 -> Resistor_SMD:R_0402_1005Metric
- TP11, TP12, TP15, TP16, TP19, TP20, TP23, TP24, TP27, TP28, TP5, TP6: footprint mmlab-footprint-library:TESTPOINT-TH_BD1.0 -> TestPoint:TestPoint_Pad_2.0x2.0mm
- U2, U3: footprint mmlab-footprint-library:TSSOP-20 -> 1mmlab_footprint:TSSOP-20
- USB1: renamed from J17; footprint Connector_IDC:IDC-Header_2x10_P2.54mm_Vertical -> Connector_PinSocket_1.27mm:PinSocket_2x10_P1.27mm_Vertical
- VDC_BUS1: renamed from TP32; footprint mmlab-footprint-library:TESTPOINT-TH_BD1.0 -> TestPoint:TestPoint_Pad_2.0x2.0mm
- VDC_BUS2: renamed from TP33; footprint mmlab-footprint-library:TESTPOINT-TH_BD1.0 -> TestPoint:TestPoint_Pad_2.0x2.0mm
- renumbered J1 to INC1, J2 to INC2
Connections:
- net -5V_ADC is gone; now on net A-5V: SPI1.17, SPI1.19
- net D12VGND is gone; now on net 12VGND: R55.1, R56.1
- net ADD4: now also P1.168 (ADD5_168); no longer P1.167 (167_ADD4)
- net ADD5: now also P1.167 (167_ADD4); no longer P1.168 (ADD5_168)
- net AD_14: now also P1.166 (AD15_166); no longer P1.165 (165_AD14)
- net AD_15: now also P1.165 (165_AD14); no longer P1.166 (AD15_166)
- net AGND: now also DI1.2 (Pin_2), U4.1 (~{OE1}), U4.15 (~{OE2}), U4.8 (GND)
- net AVDD: no longer POWER1.27
- net BootFromFlash: now also P1.120 (A1_120); no longer P1.119 (119_GP84)
- net D+5V: now also DI1.1 (Pin_1)
- net DI-1-DSP-3.3V: now also P1.96 (A13_96), U4.3 (Y1); no longer P1.95 (95_D9)
- net DI-2-DSP-3.3V: now also P1.98 (A12_98), U4.5 (Y2); no longer P1.97 (97_D8)
- net DI_1: now also U4.2 (A1)
- net DI_2: now also U4.4 (A2)
- net DSP-PWM10A: now also P1.205 (205_PWM4A); no longer P1.206 (PWM10A_206)
- net DSP-PWM10B: now also P1.207 (207_PWM4B); no longer P1.208 (PWM10B_208)
- net DSP-PWM11A: now also P1.209 (209_PWM5A); no longer P1.210 (PWM11A_210)
- net DSP-PWM11B: now also P1.211 (211_PWM5B); no longer P1.212 (PWM11B_212)
- net DSP-PWM12A: now also P1.213 (213_PWM6A); no longer P1.214 (PWM12A_214)
- net DSP-PWM12B: now also P1.215 (215_PWM6B); no longer P1.216 (PWM12B_216)
- net DSP-PWM1A: now also P1.194 (PWM7A_194); no longer P1.193 (193_PWM1A)
- net DSP-PWM1B: now also P1.196 (PWM7B_196); no longer P1.195 (195_PWM1B)
- net DSP-PWM2A: now also P1.198 (PWM8A_198); no longer P1.197 (197_PWM2A)
- net DSP-PWM2B: now also P1.200 (PWM8B_200); no longer P1.199 (199_PWM2B)
- net DSP-PWM3A: now also P1.202 (PWM9A_202); no longer P1.201 (201_PWM3A)
- net DSP-PWM3B: now also P1.204 (PWM9B_204); no longer P1.203 (203_PWM3B)
- net DSP-PWM4A: now also P1.206 (PWM10A_206); no longer P1.205 (205_PWM4A)
- net DSP-PWM4B: now also P1.208 (PWM10B_208); no longer P1.207 (207_PWM4B)
- net DSP-PWM5A: now also P1.210 (PWM11A_210); no longer P1.209 (209_PWM5A)
- net DSP-PWM5B: now also P1.212 (PWM11B_212); no longer P1.211 (211_PWM5B)
- net DSP-PWM6A: now also P1.214 (PWM12A_214); no longer P1.213 (213_PWM6A)
- net DSP-PWM6B: now also P1.216 (PWM12B_216); no longer P1.215 (215_PWM6B)
- net DSP-PWM7A: now also P1.193 (193_PWM1A); no longer P1.194 (PWM7A_194)
- net DSP-PWM7B: now also P1.195 (195_PWM1B); no longer P1.196 (PWM7B_196)
- net DSP-PWM8A: now also P1.197 (197_PWM2A); no longer P1.198 (PWM8A_198)
- net DSP-PWM8B: now also P1.199 (199_PWM2B); no longer P1.200 (PWM8B_200)
- net DSP-PWM9A: now also P1.201 (201_PWM3A); no longer P1.202 (PWM9A_202)
- net DSP-PWM9B: now also P1.203 (203_PWM3B); no longer P1.204 (PWM9B_204)
- net DSP_A_CAN_RX: now also P1.17 (17_GP19); no longer P1.18 (GP62_18)
- net DSP_A_CAN_TX: now also P1.18 (GP62_18); no longer P1.17 (17_GP19)
- net DSP_B_CAN_RX: now also P1.33 (33_GP20); no longer P1.34 (GP21_34)
- net DSP_B_CAN_TX: now also P1.34 (GP21_34); no longer P1.33 (33_GP20)
- net DSP_PWM1_~{FAULT}: now also P1.112 (A5_112); no longer P1.111 (111_D1)
- net DSP_PWM1~{_ENABL}E: now also P1.154 (GP28_154); no longer P1.153 (153_GP108)
- net DSP_PWM2_~{FAULT}: now also P1.110 (A6_110); no longer P1.109 (109_D2)
- net DSP_PWM2~{_ENABL}E: now also P1.156 (GP29_156); no longer P1.155 (155_GP93)
- net DSP_PWM3_~{FAULT}: now also P1.108 (A7_108); no longer P1.107 (107_D3)
- net DSP_PWM3~{_ENABL}E: now also P1.153 (153_GP108); no longer P1.154 (GP28_154)
- net DSP_PWM4_~{FAULT}: now also P1.106 (A8_106); no longer P1.105 (105_D4)
- net DSP_PWM4~{_ENABL}E: now also P1.155 (155_GP93); no longer P1.156 (GP29_156)
- net ECAP1_IPM_TerminalDutyU1: now also P1.83 (83_D15); no longer P1.84 (A19_84)
- net ECAP2_IPM_TerminalDutyV1: now also P1.85 (85_D14); no longer P1.86 (A18_86)
- net ECAP3_IPM_TerminalDutyW1: now also P1.87 (87_D13); no longer P1.88 (A17_88)
- net ECAP4_IPM_TerminalDutyU2: now also P1.89 (89_D12); no longer P1.90 (A16_90)
- net ECAP5_IPM_TerminalDutyV2: now also P1.91 (91_D11); no longer P1.92 (A15_92)
- net ECAP6_IPM_TerminalDutyW2: now also P1.93 (93_D10); no longer P1.94 (A14_94)
- net IPM_IU1: now also P1.188 (ADA0_188); no longer P1.187 (187_ADA1)
- net IPM_IU2: now also P1.182 (ADB0_182); no longer P1.181 (181_ADB1)
- net IPM_IU3: now also P1.172 (ADD0_172); no longer P1.171 (171_ADD1)
- net IPM_IU4: now also P1.176 (ADC2_176); no longer P1.175 (175_ADC3)
- net IPM_IV1: now also P1.185 (185_ADA3); no longer P1.186 (ADA2_186)
- net IPM_IV2: now also P1.179 (179_ADB3); no longer P1.180 (ADB2_180)
- net IPM_IV3: now also P1.169 (169_ADD2); no longer P1.170 (ADD3_170)
- net IPM_IV4: now also P1.173 (173_ADC5); no longer P1.174 (ADC4_174)
- net IPM_IW1: now also P1.186 (ADA2_186); no longer P1.185 (185_ADA3)
- net IPM_IW2: now also P1.180 (ADB2_180); no longer P1.179 (179_ADB3)
- net IPM_IW3: now also P1.170 (ADD3_170); no longer P1.169 (169_ADD2)
- net IPM_IW4: now also P1.174 (ADC4_174); no longer P1.173 (173_ADC5)
- net IPM_Temperature1: now also P1.184 (ADA4_184); no longer P1.183 (183_ADA5)
- net IPM_Temperature2: now also P1.178 (ADB4_178); no longer P1.177 (177_ADB5)
- net IPM_Temperature3: now also P1.183 (183_ADA5); no longer P1.184 (ADA4_184)
- net IPM_Temperature4: now also P1.177 (177_ADB5); no longer P1.178 (ADB4_178)
- net IPM_VDC_BUS1: now also P1.187 (187_ADA1); no longer P1.188 (ADA0_188)
- net IPM_VDC_BUS2: now also P1.181 (181_ADB1); no longer P1.182 (ADB0_182)
- net IPM_VDC_BUS3: now also P1.171 (171_ADD1); no longer P1.172 (ADD0_172)
- net IPM_VDC_BUS4: now also P1.175 (175_ADC3); no longer P1.176 (ADC2_176)
- net LED1: now also P1.12 (GP2_12); no longer P1.11 (11_GP3)
- net LED2: now also P1.11 (11_GP3); no longer P1.12 (GP2_12)
- net LED3: now also P1.14 (GP8_14); no longer P1.13 (13_GP9)
- net LED4: now also P1.13 (13_GP9); no longer P1.14 (GP8_14)
- net MQEP1A: now also P1.22 (GP97_22); no longer P1.21 (21_GP96)
- net MQEP1B: now also P1.21 (21_GP96); no longer P1.22 (GP97_22)
- net MQEP1S: now also P1.24 (GP99_24); no longer P1.23 (23_GP98)
- net MQEP1Z: now also P1.23 (23_GP98); no longer P1.24 (GP99_24)
- net MQEP2A: now also P1.26 (GP25_26); no longer P1.25 (25_GP24)
- net MQEP2B: now also P1.25 (25_GP24); no longer P1.26 (GP25_26)
- net MQEP2S: now also P1.28 (GP27_28); no longer P1.27 (27_GP26)
- net MQEP2Z: now also P1.27 (27_GP26); no longer P1.28 (GP27_28)
- net MQEP3A: now also P1.30 (GP105_30); no longer P1.29 (29_GP104)
- net MQEP3B: now also P1.29 (29_GP104); no longer P1.30 (GP105_30)
- net MQEP3S: now also P1.32 (GP107_32); no longer P1.31 (31_GP106)
- net MQEP3Z: now also P1.31 (31_GP106); no longer P1.32 (GP107_32)
- net MUSB_BZ: now also P1.51 (51_GP121); no longer P1.52 (GP111_52)
- net MUSB_DM: now also P1.45 (45_GP43); no longer P1.46 (GP42_46)
- net MUSB_DP: now also P1.52 (GP111_52); no longer P1.51 (51_GP121)
- net MUSB_EN: now also P1.46 (GP42_46); no longer P1.45 (45_GP43)
- net MUSB_FLT: now also P1.48 (GP112_48); no longer P1.47 (47_GP120)
- net MUSB_ID: now also P1.47 (47_GP120); no longer P1.48 (GP112_48)
- net MUSB_INT: now also P1.50 (GP114_50); no longer P1.49 (49_GP53)
- net MUSB_VB: now also P1.49 (49_GP53); no longer P1.50 (GP114_50)
- net QEP1_HALL_U: now also P1.61 (61_GP66); no longer P1.62 (GP68_62)
- net QEP1_HALL_V: now also P1.59 (59_GP57); no longer P1.60 (GP94_60)
- net QEP1_HALL_W: now also P1.57 (57_GP30); no longer P1.58 (GP17_58)
- net QEP2_HALL_U: now also P1.67 (67_GP127); no longer P1.68 (GP115_68)
- net QEP2_HALL_V: now also P1.65 (65_GP116); no longer P1.66 (GP32_66)
- net QEP2_HALL_W: now also P1.63 (63_GP131); no longer P1.64 (GP67_64)
- net QEP3_HALL_U: now also P1.69 (69_GP128); no longer P1.70 (GP117_70)
- net QEP3_HALL_V: now also P1.71 (71_GP126); no longer P1.72 (GP130_72)
- net QEP3_HALL_W: now also P1.73 (73_GP95); no longer P1.74 (GP54_74)
- net SPI B MI HS: now also P1.148 (GP143_148); no longer P1.147 (147_GP64)
- net SPI B MO HS: now also P1.146 (GP65_146); no longer P1.145 (145_GP63)
- net SPI_A_CK_HS: now also P1.43 (43_GP61); no longer P1.44 (GP60_44)
- net SPI_A_MI_HS: now also P1.78 (GP55_78); no longer P1.77 (77_GP59)
- net SPI_A_MO_HS: now also P1.76 (GP56_76); no longer P1.75 (75_GP58)
- net SPI_B_CK_HS: now also P1.145 (145_GP63); no longer P1.146 (GP65_146)
- net SPI_C_CK_HS: now also P1.88 (A17_88); no longer P1.87 (87_D13)
- net SPI_C_MI_HS: now also P1.86 (A18_86); no longer P1.85 (85_D14)
- net SPI_C_MO_HS: now also P1.84 (A19_84); no longer P1.83 (83_D15)
- net UART_SCI_RXDA: now also P1.130 (GP110_130); no longer P1.129 (129_GP136)
- net UART_SCI_RXDB: now also P1.128 (GP113_128); no longer P1.127 (127_GP138)
- net UART_SCI_RXDC: now also P1.136 (GP140_136); no longer P1.135 (135_GP139)
- net UART_SCI_RXDD: now also P1.16 (GP142_16); no longer P1.15 (15_GP141)
- net UART_SCI_TXDA: now also P1.132 (GP123_132); no longer P1.131 (131_GP135)
- net UART_SCI_TXDB: now also P1.118 (A2_118); no longer P1.117 (117_GP137)
- net UART_SCI_TXDC: now also P1.135 (135_GP139); no longer P1.136 (GP140_136)
- net UART_SCI_TXDD: now also P1.15 (15_GP141); no longer P1.16 (GP142_16)
- net VDD: now also POWER1.27, U4.16 (VCC)
- net ~{SPI_A_STE_HS}: now also P1.44 (GP60_44); no longer P1.43 (43_GP61)
- net ~{SPI_B_STE_HS}: now also P1.147 (147_GP64); no longer P1.148 (GP143_148)
- net ~{SPI_C_STE_HS}: now also P1.90 (A16_90); no longer P1.89 (89_D12)
- net at R2.2: now also DI1.3 (Pin_3)
- net at R1.2: now also DI1.4 (Pin_4)
- no-connect marks 88 -> 97
