File: PCBProject_Extension28377dBGA/ExtensionSimple2/sheet1 - Copy.kicad_sch (KiCad schematic)
At the start: 109 parts, among them P1 TMS320F28377D-BGA-Core, P10 Header 2X2, P11 Header 2X2, P12 Header 2X2, P13 Header 6X2, P14 Header 6X2, P19 Header 2X2, P20 Header 2X2, P21 Header 2X2, P22 Header 2X2, P9 Header 2X2, Q2 FMMT618TA, U2 SN74ABT541, U3 SN74ABT541, U4 SN74HC365D

Commit message: Add ExtensionSimple2
Parts:
- removed P1: TMS320F28377D-BGA-Core, 1mmlab_footprint:DSP_240, symbol sheet1-altium-import:root_0_TMS320F28377D-BGA-Core
- added DSP1: ~, 1mmlab_footprint:DSP_240, symbol 1mmlab:TMS320F28377D-BGA-Core
Connections:
- net ADD4: now also DSP1.167 (167_ADD4)
- net ADD5: now also DSP1.168 (ADD5_168)
- net AD_14: now also DSP1.165 (165_AD14)
- net AD_15: now also DSP1.166 (AD15_166)
- net AGND: now also DSP1.10 (GND10), DSP1.157 (157_GND), DSP1.158 (GND_158), DSP1.159 (159_GND), DSP1.160 (GND_160), DSP1.161 (161_GND), DSP1.162 (GND_162), DSP1.163 (163_GND), DSP1.164 (GND_164), DSP1.189 (189_GND), DSP1.190 (GND_190), DSP1.191 (191_GND), DSP1.192 (GND_192), DSP1.217 (217_GND), DSP1.218 (GND_218), DSP1.219 (219_GND), DSP1.220 (GND_220), DSP1.7 (7_GND), DSP1.8 (GND_8), DSP1.9 (9_GND)
- net BootFromFlash: now also DSP1.119 (119_GP84)
- net D+5V: now also DSP1.1 (1_+5V), DSP1.2 (+5V_2), DSP1.3 (3_+5V), DSP1.4 (+5V_4), DSP1.5 (5_+5V), DSP1.6 (+5V_6), DSP1.81 (81+5V), DSP1.82 (+5V_82)
- net DI-1-DSP-3.3V: now also DSP1.95 (95_D9)
- net DI-2-DSP-3.3V: now also DSP1.97 (97_D8)
- net DSP-PWM10A: now also DSP1.206 (PWM10A_206)
- net DSP-PWM10B: now also DSP1.208 (PWM10B_208)
- net DSP-PWM11A: now also DSP1.210 (PWM11A_210)
- net DSP-PWM11B: now also DSP1.212 (PWM11B_212)
- net DSP-PWM12A: now also DSP1.214 (PWM12A_214)
- net DSP-PWM12B: now also DSP1.216 (PWM12B_216)
- net DSP-PWM1A: now also DSP1.193 (193_PWM1A)
- net DSP-PWM1B: now also DSP1.195 (195_PWM1B)
- net DSP-PWM2A: now also DSP1.197 (197_PWM2A)
- net DSP-PWM2B: now also DSP1.199 (199_PWM2B)
- net DSP-PWM3A: now also DSP1.201 (201_PWM3A)
- net DSP-PWM3B: now also DSP1.203 (203_PWM3B)
- net DSP-PWM4A: now also DSP1.205 (205_PWM4A)
- net DSP-PWM4B: now also DSP1.207 (207_PWM4B)
- net DSP-PWM5A: now also DSP1.209 (209_PWM5A)
- net DSP-PWM5B: now also DSP1.211 (211_PWM5B)
- net DSP-PWM6A: now also DSP1.213 (213_PWM6A)
- net DSP-PWM6B: now also DSP1.215 (215_PWM6B)
- net DSP-PWM7A: now also DSP1.194 (PWM7A_194)
- net DSP-PWM7B: now also DSP1.196 (PWM7B_196)
- net DSP-PWM8A: now also DSP1.198 (PWM8A_198)
- net DSP-PWM8B: now also DSP1.200 (PWM8B_200)
- net DSP-PWM9A: now also DSP1.202 (PWM9A_202)
- net DSP-PWM9B: now also DSP1.204 (PWM9B_204)
- net DSP_A_CAN_RX: now also DSP1.18 (GP62_18)
- net DSP_A_CAN_TX: now also DSP1.17 (17_GP19)
- net DSP_B_CAN_RX: now also DSP1.34 (GP21_34)
- net DSP_B_CAN_TX: now also DSP1.33 (33_GP20)
- net DSP_PWM1_~{FAULT}: now also DSP1.111 (111_D1)
- net DSP_PWM1~{_ENABL}E: now also DSP1.153 (153_GP108)
- net DSP_PWM2_~{FAULT}: now also DSP1.109 (109_D2)
- net DSP_PWM2~{_ENABL}E: now also DSP1.155 (155_GP93)
- net DSP_PWM3_~{FAULT}: now also DSP1.107 (107_D3)
- net DSP_PWM3~{_ENABL}E: now also DSP1.154 (GP28_154)
- net DSP_PWM4_~{FAULT}: now also DSP1.105 (105_D4)
- net DSP_PWM4~{_ENABL}E: now also DSP1.156 (GP29_156)
- net ECAP1_IPM_TerminalDutyU1: now also DSP1.84 (A19_84)
- net ECAP2_IPM_TerminalDutyV1: now also DSP1.86 (A18_86)
- net ECAP3_IPM_TerminalDutyW1: now also DSP1.88 (A17_88)
- net ECAP4_IPM_TerminalDutyU2: now also DSP1.90 (A16_90)
- net ECAP5_IPM_TerminalDutyV2: now also DSP1.92 (A15_92)
- net ECAP6_IPM_TerminalDutyW2: now also DSP1.94 (A14_94)
- net IPM_IU1: now also DSP1.187 (187_ADA1)
- net IPM_IU2: now also DSP1.181 (181_ADB1)
- net IPM_IU3: now also DSP1.171 (171_ADD1)
- net IPM_IU4: now also DSP1.175 (175_ADC3)
- net IPM_IV1: now also DSP1.186 (ADA2_186)
- net IPM_IV2: now also DSP1.180 (ADB2_180)
- net IPM_IV3: now also DSP1.170 (ADD3_170)
- net IPM_IV4: now also DSP1.174 (ADC4_174)
- net IPM_IW1: now also DSP1.185 (185_ADA3)
- net IPM_IW2: now also DSP1.179 (179_ADB3)
- net IPM_IW3: now also DSP1.169 (169_ADD2)
- net IPM_IW4: now also DSP1.173 (173_ADC5)
- net IPM_Temperature1: now also DSP1.183 (183_ADA5)
- net IPM_Temperature2: now also DSP1.177 (177_ADB5)
- net IPM_Temperature3: now also DSP1.184 (ADA4_184)
- net IPM_Temperature4: now also DSP1.178 (ADB4_178)
- net IPM_VDC_BUS1: now also DSP1.188 (ADA0_188)
- net IPM_VDC_BUS2: now also DSP1.182 (ADB0_182)
- net IPM_VDC_BUS3: now also DSP1.172 (ADD0_172)
- net IPM_VDC_BUS4: now also DSP1.176 (ADC2_176)
- net LED1: now also DSP1.11 (11_GP3)
- net LED2: now also DSP1.12 (GP2_12)
- net LED3: now also DSP1.13 (13_GP9)
- net LED4: now also DSP1.14 (GP8_14)
- net MQEP1A: now also DSP1.21 (21_GP96)
- net MQEP1B: now also DSP1.22 (GP97_22)
- net MQEP1S: now also DSP1.23 (23_GP98)
- net MQEP1Z: now also DSP1.24 (GP99_24)
- net MQEP2A: now also DSP1.25 (25_GP24)
- net MQEP2B: now also DSP1.26 (GP25_26)
- net MQEP2S: now also DSP1.27 (27_GP26)
- net MQEP2Z: now also DSP1.28 (GP27_28)
- net MQEP3A: now also DSP1.29 (29_GP104)
- net MQEP3B: now also DSP1.30 (GP105_30)
- net MQEP3S: now also DSP1.31 (31_GP106)
- net MQEP3Z: now also DSP1.32 (GP107_32)
- net MUSB_BZ: now also DSP1.52 (GP111_52)
- net MUSB_DM: now also DSP1.46 (GP42_46)
- net MUSB_DP: now also DSP1.51 (51_GP121)
- net MUSB_EN: now also DSP1.45 (45_GP43)
- net MUSB_FLT: now also DSP1.47 (47_GP120)
- net MUSB_ID: now also DSP1.48 (GP112_48)
- net MUSB_INT: now also DSP1.49 (49_GP53)
- net MUSB_VB: now also DSP1.50 (GP114_50)
- net QEP1_HALL_U: now also DSP1.62 (GP68_62)
- net QEP1_HALL_V: now also DSP1.60 (GP94_60)
- net QEP1_HALL_W: now also DSP1.58 (GP17_58)
- net QEP2_HALL_U: now also DSP1.68 (GP115_68)
- net QEP2_HALL_V: now also DSP1.66 (GP32_66)
- net QEP2_HALL_W: now also DSP1.64 (GP67_64)
- net QEP3_HALL_U: now also DSP1.70 (GP117_70)
- net QEP3_HALL_V: now also DSP1.72 (GP130_72)
- net QEP3_HALL_W: now also DSP1.74 (GP54_74)
- net SPI B MI HS: now also DSP1.147 (147_GP64)
- net SPI B MO HS: now also DSP1.145 (145_GP63)
- net SPI_A_CK_HS: now also DSP1.44 (GP60_44)
- net SPI_A_MI_HS: now also DSP1.77 (77_GP59)
- net SPI_A_MO_HS: now also DSP1.75 (75_GP58)
- net SPI_B_CK_HS: now also DSP1.146 (GP65_146)
- net SPI_C_CK_HS: now also DSP1.87 (87_D13)
- net SPI_C_MI_HS: now also DSP1.85 (85_D14)
- net SPI_C_MO_HS: now also DSP1.83 (83_D15)
- net UART_SCI_RXDA: now also DSP1.129 (129_GP136)
- net UART_SCI_RXDB: now also DSP1.127 (127_GP138)
- net UART_SCI_RXDC: now also DSP1.135 (135_GP139)
- net UART_SCI_RXDD: now also DSP1.15 (15_GP141)
- net UART_SCI_TXDA: now also DSP1.131 (131_GP135)
- net UART_SCI_TXDB: now also DSP1.117 (117_GP137)
- net UART_SCI_TXDC: now also DSP1.136 (GP140_136)
- net UART_SCI_TXDD: now also DSP1.16 (GP142_16)
- net ~{SPI_A_STE_HS}: now also DSP1.43 (43_GP61)
- net ~{SPI_B_STE_HS}: now also DSP1.148 (GP143_148)
- net ~{SPI_C_STE_HS}: now also DSP1.89 (89_D12)
