File: PCBProject_InverterFNC42060F/Kicad_inverter/inverter_V0.2/inverter_power.kicad_sch (KiCad schematic)
At the start: 83 parts, among them IC1 TLP2270_D4-LF4,E, IC2 TLP2270_D4-LF4,E, IC3 TLP2270_D4-LF4,E, J1 Conn_02x06_Top_Bottom, J10 Conn_01x06_Pin, J11 Header 2, J12 Conn_01x02_Pin, J13 Conn_01x02_Pin, J14 Header 2, J15 Header 2, J17 Header 2, J2 Conn_01x08_Pin, J3 Conn_01x08_Pin, J4 Conn_01x02_Pin, J5 Conn_01x02_Pin, J6 Header 2, J7 Header 2, J8 Header 2, J9 Header 2, Q1 FMMT618TA, Q2 FNC42060F, U2 LM2675M-5.0

Commit message: cross check of invterter
Parts:
- R22: value 1K -> 10K
Changed lines of the file:
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@@
       (effects (font (size 1.27 1.27)) (justify left bottom))
     )
-    (property "Value" "1K" (at 244.7925 228.9175 90)
+    (property "Value" "10K" (at 244.7925 228.9175 90)
       (effects (font (size 1.27 1.27)) (justify left bottom))
     )
