File: PCBProject_InverterFNC42060F/Kicad_inverter/inverter_V0.2/inverter_power.kicad_pcb (KiCad board)
At the start: 2 copper layers, 176.7 x 51 mm, 83 parts, among them IC1 TLP2270_D4-LF4,E, IC2 TLP2270_D4-LF4,E, IC3 TLP2270_D4-LF4,E, J1 Conn_02x06_Top_Bottom, J10 Conn_01x06_Pin, J11 Header 2, J12 Conn_01x02_Pin, J13 Conn_01x02_Pin, J14 Header 2, J15 Header 2, J17 Header 2, J2 Conn_01x08_Pin, J3 Conn_01x08_Pin, J4 Conn_01x02_Pin, J5 Conn_01x02_Pin, J6 Header 2, J7 Header 2, J8 Header 2, J9 Header 2, Q1 FMMT618TA, Q2 FNC42060F, U2 LM2675M-5.0

Commit message: cross check of invterter
Changed lines of the file:
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@@
     )
   )
+  (gr_poly
+    (pts
+      (xy 198.4276 27.3876)
+      (arc (start 201.288213 27.3876) (mid 199.2404 28.235832) (end 198.392168 30.283645))
+    )
+    (stroke (width 0.2) (type solid)) (fill solid) (layer "F.Cu"))
+  (gr_poly
+    (pts
+      (xy 193.574403 27.423591)
+      (arc (start 193.574403 30.284204) (mid 192.726171 28.236391) (end 190.678358 27.388159))
+    )
+    (stroke (width 0.2) (type solid)) (fill solid) (layer "F.Cu"))
   (gr_rect (start 147.5 33.95) (end 156.25 57.25)
     (stroke (width 0.15) (type default)) (fill none) (layer "B.SilkS"))
@@
   (zone (net 37) (net_name "/W") (layers "F&B.Cu") (hatch edge 0.5)
     (priority 14)
-    (connect_pads (clearance 0.25))
+    (connect_pads yes (clearance 0.25))
     (min_thickness 0.2) (filled_areas_thickness no)
     (fill yes (thermal_gap 0.3) (thermal_bridge_width 0.3))
@@
   (zone (net 35) (net_name "/U") (layers "F&B.Cu") (hatch edge 0.5)
     (priority 12)
-    (connect_pads (clearance 0.25))
+    (connect_pads yes (clearance 0.25))
     (min_thickness 0.2) (filled_areas_thickness no)
     (fill yes (thermal_gap 0.3) (thermal_bridge_width 0.3))
@@
   (zone (net 36) (net_name "/V") (layers "F&B.Cu") (hatch edge 0.5)
     (priority 13)
-    (connect_pads (clearance 0.25))
+    (connect_pads yes (clearance 0.25))
     (min_thickness 0.2) (filled_areas_thickness no)
     (fill yes (thermal_gap 0.3) (thermal_bridge_width 0.3))
