File: PCBProject_Encoder/kicad_sheet6/kicad_sheet6.kicad_sch (KiCad schematic)
At the start: 73 parts, among them J1 L77HDE15SD1CH4RHNVGA, J2 HIF3FC-10PA-2.54DSA, U1 DS3486M, U2 DS3486M, U3 SN74HC365D

Commit message: 改善编码器
Parts:
- R1, R2, R3, R4, R5, R6: footprint Resistor_SMD:R_0402_1005Metric -> Resistor_SMD:R_0805_2012Metric
Changed lines of the file:
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@@
       (effects (font (size 1.27 1.27)) (justify left bottom))
     )
-    (property "Footprint" "Resistor_SMD:R_0402_1005Metric" (at 114.3 413.6644 0)
+    (property "Footprint" "Resistor_SMD:R_0805_2012Metric" (at 114.3 413.6644 0)
       (effects (font (size 1.27 1.27)) hide)
     )
@@
       (effects (font (size 1.27 1.27)) (justify left bottom))
     )
-    (property "Footprint" "Resistor_SMD:R_0402_1005Metric" (at 111.76 284.1244 0)
+    (property "Footprint" "Resistor_SMD:R_0805_2012Metric" (at 111.76 284.1244 0)
       (effects (font (size 1.27 1.27)) hide)
     )
@@
       (effects (font (size 1.27 1.27)) (justify left bottom))
     )
-    (property "Footprint" "Resistor_SMD:R_0402_1005Metric" (at 114.3 385.7244 0)
+    (property "Footprint" "Resistor_SMD:R_0805_2012Metric" (at 114.3 385.7244 0)
       (effects (font (size 1.27 1.27)) hide)
     )
@@
       (effects (font (size 1.27 1.27)) (justify left bottom))
     )
-    (property "Footprint" "Resistor_SMD:R_0402_1005Metric" (at 114.3 441.6044 0)
+    (property "Footprint" "Resistor_SMD:R_0805_2012Metric" (at 114.3 441.6044 0)
       (effects (font (size 1.27 1.27)) hide)
     )
@@
       (effects (font (size 1.27 1.27)) (justify left bottom))
     )
-    (property "Footprint" "Resistor_SMD:R_0402_1005Metric" (at 111.76 312.0644 0)
+    (property "Footprint" "Resistor_SMD:R_0805_2012Metric" (at 111.76 312.0644 0)
       (effects (font (size 1.27 1.27)) hide)
     )
@@
       (effects (font (size 1.27 1.27)) (justify left bottom))
     )
-    (property "Footprint" "Resistor_SMD:R_0402_1005Metric" (at 111.76 340.0044 0)
+    (property "Footprint" "Resistor_SMD:R_0805_2012Metric" (at 111.76 340.0044 0)
       (effects (font (size 1.27 1.27)) hide)
     )

Commit message: 重新布线+原图备份x1
Parts:
- C1, C10, C11, C12, C13, C14, C15, C16, C17, C18, C19, C2, C20, C21, C22, C23, C24, C25, C26, C27, C28, C29, C3, C30, C31, C32, C33, C4, C5, C6, C7, C8, C9: footprint Capacitor_SMD:C_0402_1005Metric -> Capacitor_SMD:C_0805_2012Metric
- J1: footprint Connector_Dsub:DSUB-15-HD_Male_Horizontal_P2.29x1.98mm_EdgePinOffset3.03mm_Housed_MountingHolesOffset4.94mm -> Connector_Dsub:DSUB-15-HD_Female_Horizontal_P2.29x1.98mm_EdgePinOffset3.03mm_Housed_MountingHolesOffset4.94mm
- R10, R11, R12, R13, R14, R15, R16, R17, R18, R19, R20, R21, R22, R23, R24, R7, R8, R9, RK1, RK2, RK3: footprint Resistor_SMD:R_0402_1005Metric -> Resistor_SMD:R_0805_2012Metric
