File: PCBProject_Happy485/rs485_SN65HVD75_TestBoard.kicad_pcb (KiCad board)
At the start: 2 copper layers, 30 x 14.5 mm, 12 parts, among them J1 UART_CONNECT, J2 RS485_CONNECT, J3 RS485_CONNECT, U1 SN65HVD75D

Commit message: finish happy485
Parts:
- removed J2, J3: RS485_CONNECT, Connector_PinSocket_2.54mm:PinSocket_1x02_P2.54mm_Vertical
- added J4: Conn_01x06, Connector_PinHeader_2.54mm:PinHeader_1x06_P2.54mm_Vertical, F.Cu at (157.0, 85.5)
- J1: value UART_CONNECT -> Conn_01x04; footprint Connector_PinSocket_2.54mm:PinSocket_1x03_P2.54mm_Vertical -> Connector_PinHeader_2.54mm:PinHeader_1x04_P2.54mm_Vertical
- moved J1 23.9 mm to (180.7, 89.3)
- moved R7 1.25 mm to (175.7, 93.1)
- moved C1 1.13 mm to (173.3, 92.6)
Connections:
- J1 pad 1: /UART_RX -> +5V
- J1 pad 2: /UART_WR -> GND
- J1 pad 3: /UART_TX -> /RS485_B
Routing:
- net +3.3V: track 16.5 -> 14.1 mm
- net /RS485_B: track 8.78 -> 7.92 mm
- net GND: vias 14 -> 12
- added copper zone on F.Cu, net +5V
Other:
- board size 30 x 14.5 mm -> 30 x 17.1 mm
- board text added: "2024/04/10 ChenYM（○｀ 3′○）"
- board text removed: "2023/12/21 ChenYM"
