File: PCBProject_Extension28377dBGA/ExtensionSimple4/sheet1.kicad_pcb (KiCad board)
At the start: 4 copper layers, 146.6 x 101.9 mm, 338 parts, among them J1 Conn_02x05_Odd_Even, Q1 FMMT618TA, U1 SN74ABT541, U2 SN74ABT541, U3 SN74ABT541, U4 SN74ABT541, U5 ADR423ARZ

Commit message: modified uvw
Routing:
- net /IPM_IW3: track 57.1 -> 30.9 mm
- net /IPM_IU3: track 29.7 -> 54.3 mm
- net /IPM_IW1: track 38.9 -> 53.1 mm
- net /IPM_IU4: track 18.8 -> 32.2 mm
- net /IPM_IU1: track 51.3 -> 38.6 mm
- net /IPM_IU2: track 27.0 -> 39.3 mm
- net /IPM_IW2: track 39.2 -> 27.6 mm
- net /IPM_IW4: track 32.2 -> 21.3 mm
- net +12: track 352.2 -> 348.6 mm
- net -12: track 322.5 -> 320.7 mm
- net /IPM_IV3: track 38.0 -> 37.3 mm
