File: PCBProject_SPI_MAX5307_DAC/pcb5/pcb5.kicad_pcb (KiCad board)
At the start: 4 copper layers, 93.9 x 51.7 mm, 80 parts, among them IC1 MAX5725BAUP+, U1 SN74HC365D, U2 LM224DR, U3 LM224DR

Commit message: finish ExtensionSimple3
Routing:
- net Net-(BNC1-PadMH1): track 10.9 -> 11.2 mm, vias 0 -> 1
- net GNDREF: vias 29 -> 54
Changed lines of the file:
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@@
   (segment (start 107.455 72.898) (end 108.839 72.898) (width 0.25) (layer "F.Cu") (net 10))
   (segment (start 69.977 75.102) (end 69.977 74.295) (width 0.25) (layer "F.Cu") (net 10))
+  (via (at 68.657 66.451) (size 0.8) (drill 0.4) (layers "F.Cu" "B.Cu") (free) (net 10))
+  (via (at 64.637 72.281) (size 0.8) (drill 0.4) (layers "F.Cu" "B.Cu") (free) (net 10))
   (via (at 137.922 57.531) (size 0.8) (drill 0.4) (layers "F.Cu" "B.Cu") (net 10))
+  (via (at 95.647 94.421) (size 0.8) (drill 0.4) (layers "F.Cu" "B.Cu") (free) (net 10))
+  (via (at 84.587 88.101) (size 0.8) (drill 0.4) (layers "F.Cu" "B.Cu") (free) (net 10))
   (via (at 76.454 89.662) (size 0.8) (drill 0.4) (layers "F.Cu" "B.Cu") (net 10))
   (via (at 78.74 76.581) (size 0.8) (drill 0.4) (layers "F.Cu" "B.Cu") (net 10))
   (via (at 70.231 79.756) (size 0.8) (drill 0.4) (layers "F.Cu" "B.Cu") (net 10))
+  (via (at 115.177 77.191) (size 0.8) (drill 0.4) (layers "F.Cu" "B.Cu") (free) (net 10))
   (via (at 85.725 74.676) (size 0.8) (drill 0.4) (layers "F.Cu" "B.Cu") (net 10))
   (via (at 89.408 88.646) (size 0.8) (drill 0.4) (layers "F.Cu" "B.Cu") (net 10))
@@
   (via (at 100.965 78.74) (size 0.8) (drill 0.4) (layers "F.Cu" "B.Cu") (net 10))
   (via (at 77.47 79.375) (size 0.8) (drill 0.4) (layers "F.Cu" "B.Cu") (net 10))
+  (via (at 73.457 94.541) (size 0.8) (drill 0.4) (layers "F.Cu" "B.Cu") (free) (net 10))
   (via (at 118.491 88.9) (size 0.8) (drill 0.4) (layers "F.Cu" "B.Cu") (net 10))
+  (via (at 143.577 94.951) (size 0.8) (drill 0.4) (layers "F.Cu" "B.Cu") (free) (net 10))
   (via (at 123.317 87.503) (size 0.8) (drill 0.4) (layers "F.Cu" "B.Cu") (net 10))
+  (via (at 118.177 66.161) (size 0.8) (drill 0.4) (layers "F.Cu" "B.Cu") (free) (net 10))
+  (via (at 74.807 53.531) (size 0.8) (drill 0.4) (layers "F.Cu" "B.Cu") (free) (net 10))
   (via (at 143.002 89.662) (size 0.8) (drill 0.4) (layers "F.Cu" "B.Cu") (net 10))
+  (via (at 65.987 85.871) (size 0.8) (drill 0.4) (layers "F.Cu" "B.Cu") (free) (net 10))
   (via (at 100.076 81.661) (size 0.8) (drill 0.4) (layers "F.Cu" "B.Cu") (net 10))
   (via (at 105.918 76.708) (size 0.8) (drill 0.4) (layers "F.Cu" "B.Cu") (net 10))
@@
   (via (at 116.586 65.151) (size 0.8) (drill 0.4) (layers "F.Cu" "B.Cu") (net 10))
   (via (at 99.949 89.027) (size 0.8) (drill 0.4) (layers "F.Cu" "B.Cu") (net 10))
+  (via (at 119.807 97.461) (size 0.8) (drill 0.4) (layers "F.Cu" "B.Cu") (free) (net 10))
   (via (at 115.824 80.772) (size 0.8) (drill 0.4) (layers "F.Cu" "B.Cu") (net 10))
+  (via (at 79.747 78.681) (size 0.8) (drill 0.4) (layers "F.Cu" "B.Cu") (free) (net 10))
   (via (at 72.136 57.658) (size 0.8) (drill 0.4) (layers "F.Cu" "B.Cu") (net 10))
   (via (at 94.234 57.658) (size 0.8) (drill 0.4) (layers "F.Cu" "B.Cu") (net 10))
+  (via (at 97.107 53.301) (size 0.8) (drill 0.4) (layers "F.Cu" "B.Cu") (free) (net 10))
+  (via (at 118.267 62.981) (size 0.8) (drill 0.4) (layers "F.Cu" "B.Cu") (free) (net 10))
+  (via (at 86.037 91.651) (size 0.8) (drill 0.4) (layers "F.Cu" "B.Cu") (free) (net 10))
   (via (at 73.025 67.564) (size 0.8) (drill 0.4) (layers "F.Cu" "B.Cu") (net 10))
   (via (at 73.025 80.645) (size 0.8) (drill 0.4) (layers "F.Cu" "B.Cu") (net 10))
+  (via (at 117.967 69.101) (size 0.8) (drill 0.4) (layers "F.Cu" "B.Cu") (free) (net 10))
   (via (at 89.789 76.454) (size 0.8) (drill 0.4) (layers "F.Cu" "B.Cu") (net 10))
+  (via (at 87.547 66.191) (size 0.8) (drill 0.4) (layers "F.Cu" "B.Cu") (free) (net 10))
+  (via (at 62.807 86.601) (size 0.8) (drill 0.4) (layers "F.Cu" "B.Cu") (free) (net 10))
+  (via (at 118.317 82.071) (size 0.8) (drill 0.4) (layers "F.Cu" "B.Cu") (free) (net 10))
   (via (at 100.33 65.786) (size 0.8) (drill 0.4) (layers "F.Cu" "B.Cu") (net 10))
   (via (at 69.342 73.533) (size 0.8) (drill 0.4) (layers "F.Cu" "B.Cu") (net 10))
+  (via (at 100.007 87.501) (size 0.8) (drill 0.4) (layers "F.Cu" "B.Cu") (free) (net 10))
   (via (at 89.027 66.167) (size 0.8) (drill 0.4) (layers "F.Cu" "B.Cu") (net 10))
+  (via (at 119.237 53.461) (size 0.8) (drill 0.4) (layers "F.Cu" "B.Cu") (free) (net 10))
   (via (at 115.697 57.658) (size 0.8) (drill 0.4) (layers "F.Cu" "B.Cu") (net 10))
   (via (at 107.442 60.325) (size 0.8) (drill 0.4) (layers "F.Cu" "B.Cu") (net 10))
+  (via (at 62.247 81.161) (size 0.8) (drill 0.4) (layers "F.Cu" "B.Cu") (free) (net 10))
+  (via (at 96.667 84.341) (size 0.8) (drill 0.4) (layers "F.Cu" "B.Cu") (free) (net 10))
+  (via (at 141.417 52.861) (size 0.8) (drill 0.4) (layers "F.Cu" "B.Cu") (free) (net 10))
+  (via (at 62.997 84.281) (size 0.8) (drill 0.4) (layers "F.Cu" "B.Cu") (free) (net 10))
   (segment (start 58.039 67.183) (end 60.579 67.183) (width 0.5) (layer "B.Cu") (net 10))
   (segment (start 60.579 67.183) (end 60.579 69.723) (width 0.5) (layer "B.Cu") (net 10))
@@
   (segment (start 74.98 91.186) (end 78.232 91.186) (width 0.25) (layer "F.Cu") (net 17))
   (segment (start 74.091 92.075) (end 74.98 91.186) (width 0.25) (layer "F.Cu") (net 17))
+  (segment (start 72.223 92.075) (end 74.091 92.075) (width 0.25) (layer "F.Cu") (net 17))
   (segment (start 78.232 91.186) (end 79.121 92.075) (width 0.25) (layer "F.Cu") (net 17))
-  (segment (start 68.961 92.075) (end 74.091 92.075) (width 0.25) (layer "F.Cu") (net 17))
+  (segment (start 68.961 92.075) (end 71.491 92.075) (width 0.25) (layer "F.Cu") (net 17))
+  (segment (start 71.491 92.075) (end 71.857 92.441) (width 0.25) (layer "F.Cu") (net 17))
+  (segment (start 71.857 92.441) (end 72.223 92.075) (width 0.25) (layer "F.Cu") (net 17))
+  (via (at 71.857 92.441) (size 0.8) (drill 0.4) (layers "F.Cu" "B.Cu") (net 17))
   (segment (start 93.218 88.646) (end 92.138 88.646) (width 0.25) (layer "F.Cu") (net 18))
   (segment (start 93.599 88.265) (end 93.218 88.646) (width 0.25) (layer "F.Cu") (net 18))

Commit message: finish happy485
Routing:
- net Net-(BNC1-PadMH1): track 11.2 -> 11.1 mm, vias 1 -> 0
Changed lines of the file:
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@@
     (fp_line (start 1 0.625) (end 1 -0.625)
       (stroke (width 0.1) (type solid)) (layer "B.Fab"))
-    (pad "1" smd roundrect (at -0.9125 0 180) (size 1.025 1.4) (layers "B.Cu" "B.Paste" "B.Mask") (roundrect_rratio 0.243902)
+    (pad "1" smd roundrect (at -0.9125 0 180) (size 1.025 1.4) (layers "B.Cu" "B.Paste" "B.Mask") (roundrect_rratio 0.243902439)
       (net 26 "REF_3V") (pinfunction "1") (pintype "passive"))
-    (pad "2" smd roundrect (at 0.9125 0 180) (size 1.025 1.4) (layers "B.Cu" "B.Paste" "B.Mask") (roundrect_rratio 0.243902)
+    (pad "2" smd roundrect (at 0.9125 0 180) (size 1.025 1.4) (layers "B.Cu" "B.Paste" "B.Mask") (roundrect_rratio 0.243902439)
       (net 57 "Net-(RU1-Pad2)") (pinfunction "2") (pintype "passive"))
     (model "${KICAD6_3DMODEL_DIR}/Resistor_SMD.3dshapes/R_0805_2012Metric.wrl"
@@
   (segment (start 60.579 82.423) (end 60.579 79.883) (width 1) (layer "B.Cu") (net 16))
   (segment (start 55.88 58.547) (end 55.88 56.896) (width 1) (layer "B.Cu") (net 16))
-  (segment (start 74.98 91.186) (end 78.232 91.186) (width 0.25) (layer "F.Cu") (net 17))
-  (segment (start 74.091 92.075) (end 74.98 91.186) (width 0.25) (layer "F.Cu") (net 17))
-  (segment (start 72.223 92.075) (end 74.091 92.075) (width 0.25) (layer "F.Cu") (net 17))
-  (segment (start 78.232 91.186) (end 79.121 92.075) (width 0.25) (layer "F.Cu") (net 17))
-  (segment (start 68.961 92.075) (end 71.491 92.075) (width 0.25) (layer "F.Cu") (net 17))
-  (segment (start 71.491 92.075) (end 71.857 92.441) (width 0.25) (layer "F.Cu") (net 17))
-  (segment (start 71.857 92.441) (end 72.223 92.075) (width 0.25) (layer "F.Cu") (net 17))
-  (via (at 71.857 92.441) (size 0.8) (drill 0.4) (layers "F.Cu" "B.Cu") (net 17))
+  (segment (start 74.028 92.075) (end 75.142 90.961) (width 0.25) (layer "F.Cu") (net 17))
+  (segment (start 75.142 90.961) (end 78.007 90.961) (width 0.25) (layer "F.Cu") (net 17))
+  (segment (start 78.007 90.961) (end 79.121 92.075) (width 0.25) (layer "F.Cu") (net 17))
+  (segment (start 68.961 92.075) (end 74.028 92.075) (width 0.25) (layer "F.Cu") (net 17))
   (segment (start 93.218 88.646) (end 92.138 88.646) (width 0.25) (layer "F.Cu") (net 18))
   (segment (start 93.599 88.265) (end 93.218 88.646) (width 0.25) (layer "F.Cu") (net 18))

Commit message: DAC for 28388
Parts:
- removed RU1: 0R, Resistor_SMD:R_0805_2012Metric
- added C33: 104, Capacitor_SMD:C_0805_2012Metric, F.Cu at (122.0, 81.3)
- added C34: 106 25V, Capacitor_SMD:C_1206_3216Metric, F.Cu at (122.0, 78.9)
- added C35: 104, Capacitor_SMD:C_0805_2012Metric, F.Cu at (122.5, 68.7)
- added C36: 106 25V, Capacitor_SMD:C_1206_3216Metric, F.Cu at (122.7, 66.2)
- added C37: 10uF, Capacitor_SMD:C_0805_2012Metric, F.Cu at (81.4, 65.9)
- added C38: 10uF, Capacitor_SMD:C_0805_2012Metric, F.Cu at (91.4, 66.1)
- added C39: 0.1uF, Capacitor_SMD:C_0805_2012Metric, F.Cu at (93.7, 66.1)
- added G***: LOGO, LOGO, B.Cu at (125.2, 73.9)
- added U4: ADR423ARZ, SamacSys_Parts:SOIC127P600X175-8N, F.Cu at (121.4, 73.7)
- added U5: LM2662M_NOPB, SamacSys_Parts:SOIC127P600X175-8N, F.Cu at (86.4, 65.1)
- moved C26 33.6 mm to (141.7, 63.0), turned to -90 degrees
- moved R19 27.9 mm to (139.2, 62.2), turned to 0 degrees
- moved C30 24.3 mm to (75.8, 62.0), turned to 180 degrees
- moved C23 22.5 mm to (138.7, 84.2)
- moved R13 22.5 mm to (135.5, 84.2)
- moved R34 21.9 mm to (83.9, 85.0)
- moved C32 21.0 mm to (81.3, 85.8), turned to -90 degrees
- moved R28 20.5 mm to (81.0, 60.2)
- moved C31 13.9 mm to (97.8, 62.2), turned to 180 degrees
- moved C24 13.8 mm to (119.8, 62.0)
- moved C27 13.5 mm to (118.0, 85.0), turned to 0 degrees
- moved C1 12.4 mm to (67.7, 67.1), turned to 90 degrees
- moved R14 10.5 mm to (119.7, 63.6), turned to 0 degrees
- moved R33 9.72 mm to (98.5, 64.5), turned to 90 degrees
- moved C2 8.97 mm to (68.3, 71.9)
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Connections:
- net /SPISIMIA_5V renamed /SPISOMIA_5V
- net /SPI_C_CK_HS renamed /SPI_CK_HS
- net /SPI_C_MI_HS renamed /SPI_MI_HS
- net /SPI_C_MO_HS renamed /SPI_MO_HS
- net /~{SPI_C_STE_HS} renamed /~{SPI_STE_HS}
- BNC1 pad 1: Net-(BNC1-Pad1) -> /DACA
- BNC1 pad 2: /DACA -> Net-(BNC1-Pad2)
- BNC2 pad 1: Net-(BNC2-Pad1) -> /DACB
- BNC2 pad 2: /DACB -> Net-(BNC2-Pad2)
- BNC3 pad 1: Net-(BNC3-Pad1) -> /DACC
- BNC3 pad 2: /DACC -> Net-(BNC3-Pad2)
- BNC4 pad 1: Net-(BNC4-Pad1) -> /DACD
- BNC4 pad 2: /DACD -> Net-(BNC4-Pad2)
- BNC5 pad 1: Net-(BNC5-Pad1) -> /DACE
- BNC5 pad 2: /DACE -> Net-(BNC5-Pad2)
- BNC6 pad 1: Net-(BNC6-Pad1) -> /DACF
- BNC6 pad 2: /DACF -> Net-(BNC6-Pad2)
- BNC7 pad 1: Net-(BNC7-Pad1) -> /DACG
- BNC7 pad 2: /DACG -> Net-(BNC7-Pad2)
- BNC8 pad 1: Net-(BNC8-Pad1) -> /DACH
- BNC8 pad 2: /DACH -> Net-(BNC8-Pad2)
- C14 pad 1: -5V_ADC -> -5V
- C15 pad 2: -5V_ADC -> -5V
- C16 pad 1: -5V_ADC -> -5V
- C17 pad 2: -5V_ADC -> -5V
- C18 pad 1: A+5V -> D+5V
- C19 pad 1: A+5V -> D+5V
- C20 pad 2: A+5V -> D+5V
- C21 pad 2: A+5V -> D+5V
- R1 pad 2: Net-(BNC1-Pad1) -> Net-(BNC1-Pad2)
- R2 pad 2: Net-(BNC5-Pad1) -> Net-(BNC5-Pad2)
- R3 pad 2: Net-(BNC2-Pad1) -> Net-(BNC2-Pad2)
- R4 pad 2: Net-(BNC6-Pad1) -> Net-(BNC6-Pad2)
- R5 pad 2: Net-(BNC3-Pad1) -> Net-(BNC3-Pad2)
- R6 pad 2: Net-(BNC7-Pad1) -> Net-(BNC7-Pad2)
- R7 pad 2: Net-(BNC4-Pad1) -> Net-(BNC4-Pad2)
- R8 pad 2: Net-(BNC8-Pad1) -> Net-(BNC8-Pad2)
- SPI-DAC1 pad 10: -5V_ADC -> unconnected-(SPI-DAC1-Pad10)
- SPI-DAC1 pad 11: A+5V -> D+5V
- SPI-DAC1 pad 12: A+5V -> D+5V
- SPI-DAC1 pad 15: PE_GND -> unconnected-(SPI-DAC1-Pad15)
- SPI-DAC1 pad 16: PE_GND -> unconnected-(SPI-DAC1-Pad16)
- SPI-DAC1 pad 19: Net-(RU1-Pad2) -> PE_GND
- SPI-DAC1 pad 20: Net-(RU1-Pad2) -> PE_GND
- SPI-DAC1 pad 9: -5V_ADC -> unconnected-(SPI-DAC1-Pad9)
- U2 pad 11: -5V_ADC -> -5V
- U2 pad 4: A+5V -> D+5V
- U3 pad 11: -5V_ADC -> -5V
- U3 pad 4: A+5V -> D+5V
Routing:
- net PE_GND: track 245.0 -> 0.00 mm, vias 8 -> 34
- net A+5V: track 190.4 -> 0.00 mm, vias 5 -> 0
- net -5V_ADC: track 128.8 -> 0.00 mm, vias 7 -> 0
- net REF_3V: track 208.8 -> 85.2 mm, vias 9 -> 13
- net -5V: track 0.00 -> 59.2 mm, vias 0 -> 2
- net /DACB: track 38.4 -> 3.78 mm
- net /DACG: track 38.1 -> 3.50 mm
- net /DACF: track 38.0 -> 3.54 mm
- net /DACD: track 38.0 -> 4.45 mm
- net /DACE: track 38.0 -> 4.85 mm
- net /DACH: track 38.2 -> 5.44 mm
- net /DACA: track 41.8 -> 12.4 mm
- net /DACC: track 37.6 -> 10.5 mm
- net Net-(R17-Pad2): track 5.97 -> 32.8 mm
- net /SPI_CK_HS: track 43.1 -> 16.5 mm
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- added copper zone on F.Cu, net -5V
- added copper zone on B.Cu, net D+5V
- added copper zone on F.Cu, net D+5V
- added copper zone on B.Cu, net PE_GND
- added copper zone on F.Cu, net PE_GND
- added copper zone on In1.Cu, net PE_GND
- added copper zone on In2.Cu, net PE_GND
- added copper zone on B.Cu, net REF_3V
- added copper zone on F.Cu, net REF_3V
Other:
- board text added: "1"
- board text added: "2"
- board text added: "3"
- board text added: "4"
- board text added: "5"
- board text added: "6"
- board text added: "7"
- board text added: "8"
- board text added: "DAC for 28388D"
- board text added: "JLCJLCJLCJLC"
- board text added: "Meow"

Commit message: fix bugs
Routing:
- net REF_3V: track 85.2 -> 82.3 mm
Changed lines of the file:
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@@
 	(footprint "Resistor_SMD:R_0603_1608Metric"
 		(layer "F.Cu")
-		(at 114.962 80.041 180)
+		(at 114.977 80.011 180)
 		(descr "Resistor SMD 0603 (1608 Metric), square (rectangular) end terminal, IPC_7351 nominal, (Body size source: IPC-SM-782 page 72, https://www.pcb-3d.com/wordpress/wp-content/uploads/ipc-sm-782a_amendment_1_and_2.pdf), generated with kicad-footprint-generator")
 		(tags "resistor")
@@
 	(footprint "Capacitor_SMD:C_0603_1608Metric"
 		(layer "F.Cu")
-		(at 114.337 82.241 90)
+		(at 114.357 82.286 90)
 		(descr "Capacitor SMD 0603 (1608 Metric), square (rectangular) end terminal, IPC_7351 nominal, (Body size source: IPC-SM-782 page 76, https://www.pcb-3d.com/wordpress/wp-content/uploads/ipc-sm-782a_amendment_1_and_2.pdf), generated with kicad-footprint-generator")
 		(tags "capacitor")
@@
 	)
 	(segment
-		(start 99.687 84.591)
-		(end 99.537 84.441)
+		(start 115.587 84.651)
+		(end 115.587 85.041)
 		(width 0.3)
 		(layer "F.Cu")
@@
 	)
 	(segment
-		(start 115.587 84.091)
-		(end 115.587 85.041)
+		(start 113.007 84.161)
+		(end 115.097 84.161)
 		(width 0.3)
 		(layer "F.Cu")
@@
 	)
 	(segment
-		(start 115.362 83.866)
-		(end 115.587 84.091)
+		(start 99.687 84.591)
+		(end 99.537 84.441)
 		(width 0.3)
 		(layer "F.Cu")
@@
 	)
 	(segment
-		(start 113.526944 83.866)
-		(end 115.362 83.866)
-		(width 0.3)
-		(layer "F.Cu")
-		(net 22)
-	)
-	(segment
 		(start 101.087 64.441)
 		(end 100.137 64.441)
@@
 	)
 	(segment
+		(start 112.937 84.091)
+		(end 113.007 84.161)
+		(width 0.3)
+		(layer "F.Cu")
+		(net 22)
+	)
+	(segment
 		(start 116.937 64.041)
 		(end 116.937 65.241)
@@
 	)
 	(segment
+		(start 115.097 84.161)
+		(end 115.587 84.651)
+		(width 0.3)
+		(layer "F.Cu")
+		(net 22)
+	)
+	(segment
 		(start 100.987 78.791)
 		(end 100.337 79.441)
@@
 	)
 	(via
-		(at 113.526944 83.866)
+		(at 112.937 84.091)
 		(size 0.8)
 		(drill 0.4)
@@
 	)
 	(segment
-		(start 99.537 84.441)
-		(end 99.537 82.441)
+		(start 113.137 83.891)
+		(end 113.137 79.041)
 		(width 0.3)
 		(layer "B.Cu")
@@
 	)
 	(segment
-		(start 113.137 83.041)
-		(end 113.137 79.041)
+		(start 99.537 84.441)
+		(end 99.537 82.441)
 		(width 0.3)
 		(layer "B.Cu")
@@
 	)
 	(segment
-		(start 113.526944 83.866)
-		(end 113.526944 83.430944)
-		(width 0.3)
-		(layer "B.Cu")
-		(net 22)
-	)
-	(segment
-		(start 113.137 78.841)
-		(end 113.137 79.641)
-		(width 0.3)
-		(layer "B.Cu")
-		(net 22)
-	)
-	(segment
 		(start 114.537 69.041)
 		(end 114.737 69.041)
@@
 	)
 	(segment
+		(start 112.937 84.091)
+		(end 113.137 83.891)
+		(width 0.3)
+		(layer "B.Cu")
+		(net 22)
+	)
+	(segment
 		(start 100.337 79.441)
 		(end 101.337 78.441)
@@
 	)
 	(segment
-		(start 113.137 79.041)
-		(end 113.137 81.441)
-		(width 0.3)
-		(layer "B.Cu")
-		(net 22)
-	)
-	(segment
 		(start 116.437 80.041)
 		(end 114.737 80.041)
@@
 	)
 	(segment
-		(start 113.526944 83.430944)
-		(end 113.137 83.041)
-		(width 0.3)
-		(layer "B.Cu")
-		(net 22)
-	)
-	(segment
 		(start 101.688 71.392)
 		(end 101.537 71.241)
@@
 	)
 	(zone
+		(net 0)
+		(net_name "")
+		(layers "In1.Cu" "In2.Cu")
+		(hatch edge 0.5)
+		(connect_pads
+			(clearance 0)
+		)
+		(min_thickness 0.25)
+		(filled_areas_thickness no)
+		(keepout
+			(tracks allowed)
+			(vias allowed)
+			(pads allowed)
+			(copperpour not_allowed)
+			(footprints allowed)
+		)
+		(placement
+			(enabled no)
+			(sheetname "")
+		)
+		(fill
+			(thermal_gap 0.5)
+			(thermal_bridge_width 0.5)
+		)
+		(polygon
+			(pts
+				(xy 58.047 62.041) (xy 60.427 62.041) (xy 60.507 62.121) (xy 60.507 64.801) (xy 57.777 64.801) (xy 57.707 64.731)
+				(xy 57.707 62.371) (xy 58.087 61.991) (xy 58.037 62.041) (xy 58.027 62.031) (xy 58.027 61.991) (xy 58.027 62.021)
+			)
+		)
+	)
+	(zone
 		(net 10)
 		(net_name "GNDREF")
@@
 		(polygon
 			(pts
-				(xy 56.337 60.641) (xy 58.537 58.441) (xy 70.537 58.441) (xy 72.137 56.841) (xy 75.537 56.841) (xy 77.137 58.441)
+				(xy 53.627 63.351) (xy 58.537 58.441) (xy 70.537 58.441) (xy 72.137 56.841) (xy 75.537 56.841) (xy 77.137 58.441)
 				(xy 114.937 58.441) (xy 116.937 56.441) (xy 121.337 56.441) (xy 123.337 58.441) (xy 137.137 58.441)
 				(xy 138.737 56.841) (xy 142.537 56.841) (xy 144.337 58.641) (xy 144.337 88.041) (xy 142.537 89.841)
@@
 				(xy 98.937 90.841) (xy 94.137 90.841) (xy 92.137 88.841) (xy 77.537 88.841) (xy 76.337 90.041) (xy 72.737 90.041)
 				(xy 71.737 89.041) (xy 68.537 89.041) (xy 64.937 85.441) (xy 64.937 80.841) (xy 62.737 78.641) (xy 57.137 78.641)
-				(xy 56.337 77.841)
+				(xy 53.627 75.131)
+			)
+		)
+	)
+	(zone
+		(net 0)
+		(net_name "")
+		(layers "In1.Cu" "In2.Cu")
+		(hatch edge 0.5)
+		(connect_pads
+			(clearance 0)
+		)
+		(min_thickness 0.25)
+		(filled_areas_thickness no)
+		(keepout
+			(tracks allowed)
+			(vias allowed)
+			(pads allowed)
+			(copperpour not_allowed)
+			(footprints allowed)
+		)
+		(placement
+			(enabled no)
+			(sheetname "")
+		)
+		(fill
+			(thermal_gap 0.5)
+			(thermal_bridge_width 0.5)
+		)
+		(polygon
+			(pts
+				(xy 58.347 72.371) (xy 60.477 72.371) (xy 60.577 72.471) (xy 60.577 78.761) (xy 60.537 78.801) (xy 58.227 78.801)
+				(xy 58.227 72.491)
 			)
 		)
